File: control_board_with_amanero/psu.kicad_sch (KiCad schematic)
At the start: 33 parts, among them J21 220vac, K2 G6S-2, Q4 BC547, T1 9V/10VA, T3 Triad_VPP16-310, T4 9V/10VA, U10 lt3042_breakout, U11 LT1084-ADJ, U12 LT1084-ADJ, U7 TDR 2-1222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

Commit message: v2 board
Parts:
- added C16, C17: Value=22uF, Capacitor_SMD:C_1206_3216Metric_Pad1.33x1.80mm_HandSolder, symbol Device:C_Small
- added C18: Value=10nF, Capacitor_SMD:C_1206_3216Metric_Pad1.33x1.80mm_HandSolder, symbol Device:C_Small
- added C19, C20: Value=33uF Rser=350m, Capacitor_Tantalum_SMD:CP_EIA-3528-21_Kemet-B_HandSolder, symbol Device:C_Polarized
- added C21, C22, C23, C24: 0.1u, Capacitor_SMD:C_1206_3216Metric_Pad1.33x1.80mm_HandSolder, symbol Device:C_Small
- added HS1: Heatsink, Heatsink:Heatsink_Fischer_SK104-STC-STIC_35x13mm_2xDrill2.5mm, symbol Mechanical:Heatsink_Pad_2Pin
- added J15, J17, J7, J8: SEC, TerminalBlock_Philmore:TerminalBlock_Philmore_TB132_1x02_P5.00mm_Horizontal, symbol Connector_Generic:Conn_01x02
- added J5, J6: 220vac, TerminalBlock_Philmore:TerminalBlock_Philmore_TB132_1x02_P5.00mm_Horizontal, symbol Connector_Generic:Conn_01x02
- added JP4: SolderJumper_3_Open, Jumper:SolderJumper-3_P2.0mm_Open_TrianglePad1.0x1.5mm_NumberLabels, symbol Jumper:SolderJumper_3_Open
- added R16: 10K, Resistor_SMD:R_1206_3216Metric_Pad1.30x1.75mm_HandSolder, symbol Device:R
- added R19: 90.9K, Resistor_SMD:R_1206_3216Metric_Pad1.30x1.75mm_HandSolder, symbol Device:R_Small
- added R20, R21: 10k, Resistor_SMD:R_1206_3216Metric_Pad1.30x1.75mm_HandSolder, symbol Device:R_Small
- added R22: 100k, Resistor_SMD:R_1206_3216Metric_Pad1.30x1.75mm_HandSolder, symbol Device:R_Small
- added R23: 0R, Resistor_THT:R_Axial_DIN0516_L15.5mm_D5.0mm_P7.62mm_Vertical, symbol Device:R_Small
- added U14: TPS7A39, Package_SON:Texas_S-PVSON-N10_ThermalVias, symbol Regulator_Linear:TPS7A39
- C11: value C_Polarized -> 10uF
- C12, C13: value 4.7uF -> 10uF; footprint Capacitor_SMD:C_1206_3216Metric_Pad1.33x1.80mm_HandSolder -> Capacitor_THT:CP_Radial_D5.0mm_P2.00mm
- C14: value 1000uF -> 470uF
- C15: value C_Polarized -> 470uF
- C8: value C_Polarized -> 100uF
- D5: footprint Diode_THT:Diode_Bridge_32.0x5.6x17.0mm_P10.0mm_P7.5mm -> Diode_THT:Diode_Bridge_Vishay_GBU
- L1: value 12uH -> 8.2uH; footprint Inductor_SMD:L_Neosid_SM-NE127_HandSoldering -> Inductor_SMD:L_SXN_SMDRI73
- R5, R6: value R -> 100R
- R7: value R_Small -> 300R
- R8: value R_Small -> 470R
- R9: value R -> 1K
- T1: value 9V/10VA -> 6V/10VA
- U7: value TDR 2-1222 -> TDR 2-2422
Connections:
- net +12V: now also C16.2, C21.2, R19.1, U14.10 (OUTP)
- net -12V: now also C17.1, C22.1, R22.2, U14.6 (OUTN)
- net GND: now also R16.1
- net GND3: now also C16.1, C17.2, C18.1, C19.2, C20.1, C23.1, C24.2, JP4.2 (C), R20.1, U14.11 (GND), U14.4 (GND)
- net at Q4.2 (B), R9.1: now also R16.2
- net at C14.1, D3.1 (K), U11.3 (VI): now also R23.1; no longer D5.4 (+)
- net 220_L_SWITCHED: now reaches K2.8, T3.1
- net 220_L_SWITCHED: now also J5.2 (Pin_2), J6.2 (Pin_2); no longer T4.1 (AA)
- net at D6.3, T4.3 (SA): now also J7.2 (Pin_2)
- net at D6.2, T4.4 (SB): now also J7.1 (Pin_1)
- net at T3.10: now also J8.2 (Pin_2), JP4.1 (A); no longer T3.9
- net at T3.12: now also D7.3, J8.1 (Pin_1); no longer D7.2
- net at T3.7: now also D7.2, J15.2 (Pin_2); no longer D7.3
- net at C12.2, C13.2, C9.2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: now also C20.2, C24.1, U14.5 (INN)
- net at C13.1, D7.4 (+), L1.1: now also C19.1, C23.2, U14.1 (INP), U14.2 (EN)
- net at D5.2, T1.4 (SB): now also J17.1 (Pin_1)
- net at D5.3, T1.3 (SA): now also J17.2 (Pin_2)
- net 220VAC_Raw_1 renamed 220_L_RAW
- net 220VAC_Raw_2 renamed 220_N
- net 220_N: now also J5.1 (Pin_1), J6.1 (Pin_1); no longer T3.6, T4.2 (AB)
- new net: C21.1, R19.2, R20.2, U14.9 (FBP)
- new net: R21.1, U14.8 (BUF)
- new net: C22.2, R21.2, R22.1, U14.7 (FBN)
- new net: D5.4 (+), R23.2
- new net: J15.1 (Pin_1), JP4.3 (B), T3.9
- new net: C18.2, U14.3 (NR/SS)
- no-connect marks 0 -> 5
Other:
- moved on the sheet: D7
