File: control_board_with_amanero/control_board.kicad_sch (KiCad schematic)
At the start: 44 parts, among them J1 Conn_Coaxial_Small, J10 Rotary Enc, J11 IR Sensor, J12 LCD, J13 DAC Board, J14 Amanero board, J16 UART to RPI4, J19 Muted out L, J2 Conn_Coaxial_Small, J20 Muted out R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

Commit message: add readme
Other:
- note removed: "Konektor 1 - RW - MOSI - GPIO10 2 - GND - trenutno povezano na 20,1,14 3 - trenutno nije povezano ali moze za +5V - VDD - napajanje kola 4 - rst - RST - GPIO25 5 - E - SCLK - GPIO11 6 - RS - GPI08 Trenutno van konektora: 3 - 19 - osvetljaj ekrana +5V 8 - 20 - osvetljaj ekrana GND, moze tranzistor za on/off"
Changed lines of the file:
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@@
-		)
-	)
-	(text "Konektor\n1 - RW - MOSI - GPIO10\n2 - GND - trenutno povezano na 20,1,14\n3 - trenutno nije povezano ali moze za +5V - VDD - napajanje kola\n4 - rst - RST - GPIO25\n5 - E  - SCLK - GPIO11\n6 - RS - GPI08\n\nTrenutno van konektora:\n3 - 19 - osvetljaj ekrana +5V\n8 - 20 - osvetljaj ekrana GND, moze tranzistor za on/off\n\n"
-		(exclude_from_sim no)
-		(at 34.544 63.5 0)
-		(effects
-			(font
-				(size 1.27 1.27)
-			)
-			(justify left)
 		)
 	)

Commit message: v2 board
Parts:
- removed J5, J6, J7, J8: Conn_Coaxial_Small, Connector_Coaxial:U.FL_Molex_MCRF_73412-0110_Vertical, symbol Connector:Conn_Coaxial_Small
- added H1: (no value), MountingHole:MountingHole_3.2mm_M3, symbol Mechanical:MountingHole
- added H2, H7: (no value), MountingHole:MountingHole_3.2mm_M3_Pad_TopBottom, symbol Mechanical:MountingHole_Pad
- added JP1: open_if_u13_installed, Jumper:SolderJumper-2_P1.3mm_Open_Pad1.0x1.5mm, symbol Jumper:Jumper_2_Open
- added R10, R11, R12, R13, R14, R15, R17, R18: 10K, Resistor_SMD:R_1206_3216Metric_Pad1.30x1.75mm_HandSolder, symbol Device:R
- added U13: ADuM1250, Package_SO:SOIC-8_3.9x4.9mm_P1.27mm, symbol Isolator:ADuM1250
- H3, H4, H5, H6: value MountingHole -> (none)
- R1, R4: value R -> 1K
- R2: value R -> 10K
- R3: value R -> 100R
- U2, U3: value 74LS573 -> 74AC573
- U5: value ADuM1400xRW -> ADuM1250; footprint Package_SO:SOIC-16W_7.5x10.3mm_P1.27mm -> Package_SO:SOIC-8_3.9x4.9mm_P1.27mm; symbol Isolator:ADuM1400xRW -> Isolator:ADuM1250
- U6: value ADuM1400xRW -> IL715E; footprint Package_SO:SOIC-16W_7.5x10.3mm_P1.27mm -> MyLibrary:SOIC16_WIDE_NVE; symbol Isolator:ADuM1400xRW -> NVE IL751E:IL715E
Connections:
- net AMANERO_3.3V_OUT: now also C4.2, J14.10 (Pin_10); no longer C4.1
- net DAC_3.3V_OUT: now also J13.11 (Pin_11), U5.8 (VDD2), JP1.2 (B), R13.1, R14.1, R15.1, U13.8 (VDD2); no longer U5.10 (VE2), U5.16 (VDD2), U6.10 (VE2)
- net DAC_I2C_SCL: now also U5.3 (SCL1), R11.2; no longer U5.4 (VIB)
- net DAC_I2C_SCL_ISO: now also U5.6 (SCL2), R14.2; no longer U5.13 (VOB)
- net DAC_I2C_SDA: now also U5.2 (SDA1), R10.2; no longer U5.3 (VIA)
- net DAC_I2C_SDA_ISO: now also U5.7 (SDA2), R13.2; no longer U5.14 (VOA)
- net DAC_I2S_LR: now also U3.17 (Q2), U6.4 (IN2); no longer U3.15 (Q4), U6.5 (VIC)
- net DAC_I2S_LR_B: now also J14.5 (Pin_5), U3.4 (D2); no longer J14.4 (Pin_4), U3.6 (D4)
- net DAC_I2S_LR_ISO: now also U6.13 (OUT2); no longer U6.12 (VOC)
- net DAC_I2S_SCK: now also U3.15 (Q4), U6.5 (IN3); no longer U3.17 (Q2), U6.4 (VIB)
- net DAC_I2S_SCK_B: now also J14.4 (Pin_4), U3.6 (D4); no longer J14.5 (Pin_5), U3.4 (D2)
- net DAC_I2S_SCK_ISO: now also U6.12 (OUT3); no longer U6.13 (VOB)
- net DAC_PDN_CTRL: now also R12.2, U13.3 (SCL1); no longer U5.5 (VIC)
- net GND: now also C3.1, C4.1, J12.10 (Pin_10), J12.9 (Pin_9), U5.4 (GND1), H2.1, H7.1, R17.1, R18.1, U13.4 (GND1); no longer C3.2, C4.2, U4.42 (GND), U5.2 (GND1), U5.8 (GND1)
- net GND3: now also U5.5 (GND2), U13.5 (GND2); no longer U5.12 (VOC), U5.15 (GND2), U5.9 (GND2)
- net PICO_3.3V_OUT: now also C3.2, R10.1, R11.1, R12.1, U13.1 (VDD1); no longer C3.1
- net LCD_SPI_RS/DC: now reaches J12.7 (Pin_7)
- net LCD_SPI_RS/DC: now also U4.10 (GPIO7)
- net LCD_BLK_GND: now reaches J12.8 (Pin_8), Q1.1 (C)
- net DAC_PDN_CTRL_ISO: now reaches J13.15 (Pin_15)
- net DAC_PDN_CTRL_ISO: now also JP1.1 (A), R15.2, U13.6 (SCL2)
- net at Q1.2 (B), R1.2: now also R18.2
- net at Q3.2 (B), R4.2: now also R17.2
- no-connect marks 0 -> 28
Other:
- note added: "Audio out mute relay"
- note added: "I2C Isolator"
- note added: "I2S Isolator"
- note added: "I2S Switch"
- note added: "IR and Rot. Enc."
- note added: "MCU"
- note added: "TODO: - disconnect vbus and vsys of pico"
- note removed: "1 - GND 2 - MCLK 3 - GND 4 - LRCK/DSD2 5 - GND 6 - SCK/BCK/CLK 7 - GND 8 - SD(DATA)/DSD1 9 - GND 10 - GND 11 - +3.3v out 12 - +3.3V out 13,14 - not connected 15 - RST 16 - GND 17 - GND 18 - I2C - SCL 19 - GND 20 - I2C SDA"
- note removed: "1 - MCLK 2 - LRCK 3 - BCLK 4 - SD 5 - GND 6 - NC 7 - GND 8 - +5V"
- note removed: "Amanero version"
- note removed: "TOS board"
- moved on the sheet: C1, C2, C3, C4, C5, C6, D1, D2, H3, H4, H5, H6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

Commit message: add gerber and bom files
Parts:
- H1, H2, H3, H4, H5, H6, H7: value (none) -> ~
Changed lines of the file:
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@@
 			)
 		)
-		(property "Value" ""
+		(property "Value" "~"
 			(at 57.15 87.6299 0)
 			(effects
@@
 			)
 		)
-		(property "Value" ""
+		(property "Value" "~"
 			(at 31.75 105.3521 0)
 			(effects
@@
 			)
 		)
-		(property "Value" ""
+		(property "Value" "~"
 			(at 57.15 102.8699 0)
 			(show_name yes)
@@
 			)
 		)
-		(property "Value" ""
+		(property "Value" "~"
 			(at 57.15 113.0299 0)
 			(effects
@@
 			)
 		)
-		(property "Value" ""
+		(property "Value" "~"
 			(at 31.75 96.4621 0)
 			(effects
@@
 			)
 		)
-		(property "Value" ""
+		(property "Value" "~"
 			(at 31.75 87.5721 0)
 			(effects
@@
 			)
 		)
-		(property "Value" ""
+		(property "Value" "~"
 			(at 31.75 113.0299 0)
 			(show_name yes)
